File: workspace/eagle/SCD-Redesign/scd_v2.sch (EAGLE design)
At the start: 21 parts, among them J1 AVR_SPI_PRG_6PTH, U2 ATMEGA328P_TQFP

Commit message: eagle files uploaded
Parts:
- C4, C5: device rcl:CPOL-EU153CLV-0605 -> resistor:CPOL-EUTT2D7
Changed lines of the file:
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@@
 <part name="R8" library="resistor" deviceset="R-EU_" device="R0805" value="4,7k"/>
 <part name="JP1" library="pinhead" library_urn="urn:adsk.eagle:library:325" deviceset="PINHD-1X3" device="/90" package3d_urn="urn:adsk.eagle:package:22459/1"/>
-<part name="C4" library="rcl" library_urn="urn:adsk.eagle:library:334" deviceset="CPOL-EU" device="153CLV-0605" package3d_urn="urn:adsk.eagle:package:23398/1"/>
-<part name="C5" library="rcl" library_urn="urn:adsk.eagle:library:334" deviceset="CPOL-EU" device="153CLV-0605" package3d_urn="urn:adsk.eagle:package:23398/1"/>
+<part name="C4" library="resistor" library_urn="urn:adsk.eagle:library:348" deviceset="CPOL-EU" device="TT2D7" package3d_urn="urn:adsk.eagle:package:25793/1"/>
+<part name="C5" library="resistor" library_urn="urn:adsk.eagle:library:348" deviceset="CPOL-EU" device="TT2D7" package3d_urn="urn:adsk.eagle:package:25793/1"/>
 <part name="GND9" library="supply1" deviceset="GND" device=""/>
 <part name="GND10" library="supply1" deviceset="GND" device=""/>
@@
 <text x="-60.96" y="81.28" size="1.778" layer="91">A1</text>
 <text x="-60.96" y="78.74" size="1.778" layer="91">B2</text>
-<text x="-60.96" y="76.2" size="1.778" layer="91">B1</text>
+<text x="-58.42" y="71.12" size="1.778" layer="91">B1</text>
 </plain>
 <instances>
@@
 <wire x1="12.7" y1="78.74" x2="12.7" y2="15.24" width="0.1524" layer="91"/>
 <wire x1="12.7" y1="15.24" x2="30.48" y2="15.24" width="0.1524" layer="91"/>
-</segment>
-</net>
+<label x="-66.04" y="71.12" size="1.778" layer="95"/>
+<label x="-53.34" y="78.74" size="1.778" layer="95"/>
+</segment>
+</net>
